Commit message: fix: rotate Pika gripper base by Ry(-pi/2) to align with arm chain

File: src/nero_webapp/static/nero_with_gripper.urdf (robot description, URDF)
Before this commit: robot nero, 13 links, 12 joints
Joints:
- joint gripper_base_joint: origin xyz=0 0 0.0055 rpy=0 0 0 -> xyz=0 0 0.0055 rpy=0 -1.5708 0

Commit message: fix: add 180° roll to flip Pika camera facing up

File: src/nero_webapp/static/nero_with_gripper.urdf (robot description, URDF)
Before this commit: robot nero, 13 links, 12 joints
Joints:
- joint gripper_base_joint: origin xyz=0 0 0.0055 rpy=0 -1.5708 0 -> xyz=0 0 0.0055 rpy=3.1416 -1.5708 0
