Commit message: feat: replace AgileX gripper with official Pika gripper URDF + meshes
Adds pika_gripper_description package (STL meshes + URDF from
agilexrobotics/pika_ros) and updates nero_with_gripper.urdf to use
the Pika's SolidWorks-exported masses and geometry:

  gripper_base: 0.45 kg → 0.19 kg (correct for Pika)
  gripper fingers: 0.025 → 0.034 kg each
  joint axes: Z → Y (Pika's actual prismatic direction)
  meshes: DAE (agx_arm) → STL (pika_gripper)

This fixes gravity comp over-estimation at the tip (~0.26 kg
excess mass removed) and gives the 3D rendering the actual Pika
geometry instead of the AgileX standard gripper.

Webapp serves Pika meshes via /pkg/pika_gripper_description/.
URDFLoader package map updated. Jaw animation signs adjusted for
the Y-axis prismatic convention.

Co-Authored-By: Claude Opus 4.6 (1M context) <noreply@anthropic.com>

File: src/nero_webapp/static/nero_with_gripper.urdf (robot description, URDF)
Before this commit: robot nero, 13 links, 12 joints
Links:
- link gripper_base: mass 0.45 -> 0.18972; geometry collision mesh filename=package://pika_gripper_description/meshes/gripper_base_link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; visual mesh filename=package://pika_gripper_description/meshes/gripper_base_link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
- link gripper_link1: mass 0.025 -> 0.033674; geometry collision mesh filename=package://pika_gripper_description/meshes/gripper_left_link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; visual mesh filename=package://pika_gripper_description/meshes/gripper_left_link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
- link gripper_link2: mass 0.025 -> 0.033674; geometry collision mesh filename=package://pika_gripper_description/meshes/gripper_right_lin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; visual mesh filename=package://pika_gripper_description/meshes/gripper_right_lin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
Joints:
- joint gripper_joint1: axis 0 0 1 -> 0 1 0; limit lower=0 upper=0.05 effort=10 velocity=3 -> lower=-0.05 upper=0 effort=100 velocity=5; origin xyz=0 0 0.1358 rpy=1.5707963 0 3.1415926 -> xyz=0.0815 0.08851 0.0064182 rpy=0 0 0
- joint gripper_joint2: axis 0 0 -1 -> 0 1 0; limit lower=-0.05 upper=0 effort=10 velocity=3 -> lower=0 upper=0.05 effort=100 velocity=5; origin xyz=0 0 0.1358 rpy=1.5707963 0 0 -> xyz=0.0815 -0.088529 0.0064182 rpy=0 0 0

Commit message: feat(quest_leader): switch EE link from gripper_flange to gripper_tip
Add a virtual gripper_tip link to nero_with_gripper.urdf mirroring
curobo_ik_ros/robots/nero/urdf/nero_single_isaac.urdf (parent
gripper_base, xyz 0 0 0.185). FK and the cuRobo IK now solve to the
same frame, so target ↔ ghost ↔ commanded joints are consistent.

Operationally: tip is what the operator visually maps "my hand goes
here" to (between the fingertips), not the flange ~10 cm behind.
Recalibration is required on first launch — the calibration EE pose
shifts forward by the flange→tip offset.

Co-Authored-By: Claude Opus 4.7 <noreply@anthropic.com>

File: src/nero_webapp/static/nero_with_gripper.urdf (robot description, URDF)
Before this commit: robot nero, 13 links, 12 joints
Links:
- added link gripper_tip, mass 0.001
Joints:
- added joint gripper_tip_joint: type fixed, parent gripper_base, child gripper_tip, origin xyz=0 0 0.185 rpy=0 0 0

Commit message: fix(urdf): align gripper_base_joint rpy with cuRobo's URDF
curobo_ik_ros/robots/nero/urdf/nero_single_isaac.urdf has
gripper_base_joint rpy="0 0 0"; ours had "3.1416 -1.5708 0". With
gripper_tip at (0,0,0.185) in gripper_base, that disagreement put
OUR tip at flange-local (0.185, 0, 0.0055) and cuRobo's at
(0, 0, 0.24) — ~18 cm apart in flange frame.

Effect: our FK reports an EE pose, we send target = FK + delta to
cuRobo, cuRobo solves for ITS tip to land there. The returned joint
angles place cuRobo's tip at the target but our tip ends up offset
and rotated, which manifested as IK convergence pain and visibly
wrong end-effector tracking.

Trade-off: Pika finger meshes display in a different orientation in
RViz/webapp 3D, but joint commands sent to the arm are now correct.
The dual_arm xacro (visualization-only) is unchanged.

Co-Authored-By: Claude Opus 4.7 <noreply@anthropic.com>

File: src/nero_webapp/static/nero_with_gripper.urdf (robot description, URDF)
Before this commit: robot nero, 14 links, 13 joints
Joints:
- joint gripper_base_joint: origin xyz=0 0 0.0055 rpy=3.1416 -1.5708 0 -> xyz=0 0 0.0055 rpy=0 0 0

Commit message: revert "fix(urdf): align gripper_base_joint rpy with cuRobo's URDF"
This reverts 5a9c3e1. Wrong direction — our URDF correctly models the
physical Pika mount (fingers along flange +X); cuRobo's URDF has
gripper_base at identity and is the inaccurate one. Aligning ours to
cuRobo's broke our FK / ghost visualization. The proper fix is on
the cuRobo side: change nero_single_isaac.urdf's gripper_base_joint
rpy to match ours so cuRobo's gripper_tip lands at the real
physical tip.

Co-Authored-By: Claude Opus 4.7 <noreply@anthropic.com>

File: src/nero_webapp/static/nero_with_gripper.urdf (robot description, URDF)
Before this commit: robot nero, 14 links, 13 joints
Joints:
- joint gripper_base_joint: origin xyz=0 0 0.0055 rpy=0 0 0 -> xyz=0 0 0.0055 rpy=3.1416 -1.5708 0

Commit message: viz(urdf): add a red sphere marker on gripper_tip
The link was invisible before (purely a kinematic frame). Adds a
12 mm bright-red sphere at the link origin so the operator can SEE
where FK / IK is aiming when judging whether the model matches the
physical fingertip. Sphere is visual-only — no collision, negligible
inertia.

Co-Authored-By: Claude Opus 4.7 <noreply@anthropic.com>

File: src/nero_webapp/static/nero_with_gripper.urdf (robot description, URDF)
Before this commit: robot nero, 14 links, 13 joints
Links:
- link gripper_tip: geometry visual sphere radius=0.012

Commit message: fix(urdf): gripper_tip offset along gripper_base +X, not +Z
Our gripper_base is rotated rpy=(pi, -pi/2, 0) relative to flange,
so the Pika fingers physically extend along gripper_base's local +X
(gripper_joint1/2 origins are ~(0.08, ±0.09, 0.006) in gripper_base,
along +X). The previous (0, 0, 0.185) was copied from cuRobo's URDF
where gripper_base is at identity and +Z is correct — applied to
our rotated gripper_base, that landed the marker 18 cm in the wrong
direction (perpendicular to the fingers, "above" the gripper at the
home pose).

Switching to (0.185, 0, 0) puts the marker between the fingertips
in our URDF and lands at the same flange-frame point as cuRobo's
(0, 0, 0.185) lands when their gripper_base sits at identity — i.e.
the IK solver and our FK still agree on what gripper_tip means.

Co-Authored-By: Claude Opus 4.7 <noreply@anthropic.com>

File: src/nero_webapp/static/nero_with_gripper.urdf (robot description, URDF)
Before this commit: robot nero, 14 links, 13 joints
Joints:
- joint gripper_tip_joint: origin xyz=0 0 0.185 rpy=0 0 0 -> xyz=0.185 0 0 rpy=0 0 0
