Commit message: fix: set arm spacing to 185mm to match physical torso

File: src/nero_dual_description/urdf/two_nero.urdf.xacro (robot description, xacro)
@@ -13,5 +13,5 @@
   <!-- ===== Mount geometry (edit to match your physical rig) ===== -->
   <xacro:property name="torso_depth"       value="0.10"/>  <!-- X size -->
-  <xacro:property name="torso_width"       value="0.30"/>  <!-- Y size -->
+  <xacro:property name="torso_width"       value="0.185"/>  <!-- Y size -->
   <xacro:property name="torso_height"      value="0.60"/>  <!-- Z size -->
   <xacro:property name="shoulder_y_offset" value="${torso_width / 2.0}"/>
