Commit message: refactor: single source of truth for torso dimensions
Torso width/depth/height are now launch arguments that flow to
both the xacro (URDF model for robot_state_publisher) AND the
webapp node (3D rendering via /torso_config endpoint). JS fetches
the dimensions at boot instead of using hardcoded constants.

Change the torso width: pass torso_width:=0.20 to the launch
command. Both the URDF and the 3D view update automatically.

Co-Authored-By: Claude Opus 4.6 (1M context) <noreply@anthropic.com>

File: src/nero_dual_description/urdf/two_nero.urdf.xacro (robot description, xacro)
@@ -11,8 +11,13 @@
 <robot name="two_nero" xmlns:xacro="http://www.ros.org/wiki/xacro">
   <xacro:include filename="$(find nero_dual_description)/urdf/nero_arm_macro.xacro"/>
-  <!-- ===== Mount geometry (edit to match your physical rig) ===== -->
-  <xacro:property name="torso_depth"       value="0.10"/>  <!-- X size -->
-  <xacro:property name="torso_width"       value="0.185"/>  <!-- Y size -->
-  <xacro:property name="torso_height"      value="0.60"/>  <!-- Z size -->
+  <!-- ===== Mount geometry — set via launch args so there's one
+       source of truth (the launch file) for both the URDF and the
+       webapp's 3D rendering. ===== -->
+  <xacro:arg name="torso_depth"  default="0.10"/>
+  <xacro:arg name="torso_width"  default="0.185"/>
+  <xacro:arg name="torso_height" default="0.60"/>
+  <xacro:property name="torso_depth"       value="$(arg torso_depth)"/>
+  <xacro:property name="torso_width"       value="$(arg torso_width)"/>
+  <xacro:property name="torso_height"      value="$(arg torso_height)"/>
   <xacro:property name="shoulder_y_offset" value="${torso_width / 2.0}"/>
   <xacro:property name="shoulder_z"        value="${torso_height - 0.05}"/>

Commit message: feat(mount): set inter-arm spacing to 112.6 mm and add 20° shoulder tilt
Real hardware mounts the two arms 112.6 mm apart with each shoulder
rolled ±20° about its own +X axis. Plumbs a new shoulder_tilt_deg
launch arg through the xacro, robot_state_publisher, webapp
/torso_config, and the three.js render so the URDF (used by Pinocchio
IK) and the browser 3D view stay aligned.

Defaults: torso_width 0.185 → 0.1126, shoulder_tilt_deg 20.0.

Co-Authored-By: Claude Opus 4.7 <noreply@anthropic.com>

File: src/nero_dual_description/urdf/two_nero.urdf.xacro (robot description, xacro)
@@ -14,16 +14,22 @@
        source of truth (the launch file) for both the URDF and the
        webapp's 3D rendering. ===== -->
-  <xacro:arg name="torso_depth"  default="0.10"/>
-  <xacro:arg name="torso_width"  default="0.185"/>
-  <xacro:arg name="torso_height" default="0.60"/>
+  <xacro:arg name="torso_depth"       default="0.10"/>
+  <xacro:arg name="torso_width"       default="0.1126"/>
+  <xacro:arg name="torso_height"      default="0.60"/>
+  <xacro:arg name="shoulder_tilt_deg" default="20.0"/>
   <xacro:property name="torso_depth"       value="$(arg torso_depth)"/>
   <xacro:property name="torso_width"       value="$(arg torso_width)"/>
   <xacro:property name="torso_height"      value="$(arg torso_height)"/>
+  <xacro:property name="shoulder_tilt_deg" value="$(arg shoulder_tilt_deg)"/>
+  <xacro:property name="shoulder_tilt"     value="${shoulder_tilt_deg * pi / 180.0}"/>
   <xacro:property name="shoulder_y_offset" value="${torso_width / 2.0}"/>
   <xacro:property name="shoulder_z"        value="${torso_height - 0.05}"/>
   <!-- Roll each base outward so the arm's +Z axis points along ±Y instead
-       of +Z. -pi/2 for the left shoulder, +pi/2 for the right. -->
-  <xacro:property name="left_shoulder_rpy"  value="${-pi / 2} 0 0"/>
-  <xacro:property name="right_shoulder_rpy" value="${ pi / 2} 0 0"/>
+       of +Z. ±pi/2 gets the arms horizontal; shoulder_tilt adds a roll
+       around the arm's own +X axis (the shoulder "cant" of the real
+       mount). Since the first rotation is itself around X, adding to the
+       same roll composes cleanly with no axis remapping. -->
+  <xacro:property name="left_shoulder_rpy"  value="${-pi / 2 - shoulder_tilt} 0 0"/>
+  <xacro:property name="right_shoulder_rpy" value="${ pi / 2 + shoulder_tilt} 0 0"/>
   <!-- ===== World + torso ===== -->
   <link name="world"/>

Commit message: fix(dual_nero): align xacro with main.js's +X=right, +Y=front convention
The two_nero xacro was using +Y as the lateral axis (right arm at
-Y) while main.js and the axes-helper labels use +X. That mismatch
meant the URDF TF tree described the robot in a different frame
than the viz, which is why the quest-leader IK target didn't land
on the drawn rings even after transforming dp through R_mount.

Changes to two_nero.urdf.xacro:
  - shoulder_y_offset → shoulder_x_offset; lateral separation now
    along world X (right=+X, left=-X).
  - Torso box dims reordered to (width, depth, height) so `width`
    is lateral and `depth` is front-back, matching main.js.
  - Shoulder rpy:
      right: (π + tilt, -π/2, 0)
      left : (   -tilt, -π/2, 0)
    These produce the same rotation matrices as main.js's intrinsic
    Rx(π)·Ry(π/2)·Rx(+tilt) / Ry(-π/2)·Rx(-tilt). Verified
    numerically. Gravity in each base_link is (-9.81, 0, 0), which
    matches the existing gravity_comp launch arg unchanged.

Also simplified quest_leader_node's R_mount to build from the
xacro rpy triple directly (scipy extrinsic 'xyz'), since URDF and
viz now agree — one authoritative formula.

No change to gravity_comp, webapp_node, main.js (main.js already
used this convention).

Co-Authored-By: Claude Opus 4.7 <noreply@anthropic.com>

File: src/nero_dual_description/urdf/two_nero.urdf.xacro (robot description, xacro)
@@ -23,13 +23,25 @@
   <xacro:property name="shoulder_tilt_deg" value="$(arg shoulder_tilt_deg)"/>
   <xacro:property name="shoulder_tilt"     value="${shoulder_tilt_deg * pi / 180.0}"/>
-  <xacro:property name="shoulder_y_offset" value="${torso_width / 2.0}"/>
+  <!-- World convention (matches the webapp's three.js scene and its
+       axes-helper labels): +X = right, +Y = front, +Z = up. Lateral
+       separation is along X, front-back along Y. -->
+  <xacro:property name="shoulder_x_offset" value="${torso_width / 2.0}"/>
   <xacro:property name="shoulder_z"        value="${torso_height - 0.05}"/>
-  <!-- Roll each base outward so the arm's +Z axis points along ±Y instead
-       of +Z. ±pi/2 gets the arms horizontal; shoulder_tilt adds a roll
-       around the arm's own +X axis (the shoulder "cant" of the real
-       mount). Since the first rotation is itself around X, adding to the
-       same roll composes cleanly with no axis remapping. -->
-  <xacro:property name="left_shoulder_rpy"  value="${-pi / 2 - shoulder_tilt} 0 0"/>
-  <xacro:property name="right_shoulder_rpy" value="${ pi / 2 + shoulder_tilt} 0 0"/>
+  <!-- Mount rotation must match main.js::buildArms() so the URDF's TF
+       tree and the webapp's 3D scene describe the same physical
+       orientation. main.js applies (intrinsic, in order):
+         right: rotation.set(π, π/2, 0) then rotateX(+tilt)
+                →  Rx(π) · Ry(π/2) · Rx(+tilt)
+         left : rotation.y = -π/2     then rotateX(-tilt)
+                →  Ry(-π/2) · Rx(-tilt)
+       URDF rpy is extrinsic xyz (matrix = Rz(y)·Ry(p)·Rx(r)); the
+       equivalent rpy triples that produce those matrices are:
+         right: ( π + tilt, -π/2, 0 )
+         left : (   -tilt , -π/2, 0 )
+       Verified by multiplying out both forms at arbitrary tilt.
+       Gravity in base_link is (-9.81, 0, 0) for both arms under this
+       mount, matching the gravity_comp launch arg. -->
+  <xacro:property name="right_shoulder_rpy" value="${ pi + shoulder_tilt} ${-pi / 2} 0"/>
+  <xacro:property name="left_shoulder_rpy"  value="${    -shoulder_tilt} ${-pi / 2} 0"/>
   <!-- ===== World + torso ===== -->
   <link name="world"/>
@@ -38,5 +50,5 @@
       <origin xyz="0 0 ${torso_height / 2}" rpy="0 0 0"/>
       <geometry>
-        <box size="${torso_depth} ${torso_width} ${torso_height}"/>
+        <box size="${torso_width} ${torso_depth} ${torso_height}"/>
       </geometry>
       <material name="torso_grey">
@@ -47,5 +59,5 @@
       <origin xyz="0 0 ${torso_height / 2}" rpy="0 0 0"/>
       <geometry>
-        <box size="${torso_depth} ${torso_width} ${torso_height}"/>
+        <box size="${torso_width} ${torso_depth} ${torso_height}"/>
       </geometry>
     </collision>
@@ -66,5 +78,5 @@
     <parent link="torso_base"/>
     <child  link="left_shoulder_mount"/>
-    <origin xyz="0 ${ shoulder_y_offset} ${shoulder_z}"
+    <origin xyz="${-shoulder_x_offset} 0 ${shoulder_z}"
             rpy="${left_shoulder_rpy}"/>
   </joint>
@@ -73,5 +85,5 @@
     <parent link="torso_base"/>
     <child  link="right_shoulder_mount"/>
-    <origin xyz="0 ${-shoulder_y_offset} ${shoulder_z}"
+    <origin xyz="${ shoulder_x_offset} 0 ${shoulder_z}"
             rpy="${right_shoulder_rpy}"/>
   </joint>
